Commit message: update

File: orne_description/urdf/gamma/orne_gamma.urdf.xacro (robot description, xacro)
@@ -8,4 +8,5 @@
   <xacro:include filename="$(find orne_description)/urdf/gamma/orne_gamma.gazebo"/>
   <xacro:include filename="$(find orne_description)/urdf/sensors/hokuyo.urdf.xacro"/>
+  <xacro:include filename="$(find orne_description)/urdf/gamma/orne_gamma_caster_fix.urdf.xacro"/>
   <!--Base Footprint-->
   <link name="base_footprint" />
@@ -32,5 +33,5 @@
       </geometry>
     </collision>
-     <collision name="collision">
+     <!-- <collision name="collision">
       <origin xyz="0.15 0.0 -0.075" rpy="1.57 0.0 0.0"/>
       <geometry>
@@ -43,5 +44,5 @@
         <cylinder  length="0.03" radius="0.04625"/>
       </geometry>
-    </visual>
+    </visual> -->
     <!-- <inertial>
       <mass value="20" />
@@ -52,5 +53,6 @@
     <mass value="15" />
     <origin xyz="0 0 0" rpy="0 0 0"/>
-    <inertia ixx="1" ixy="0" ixz="0" iyy="1" iyz="0" izz="1" />
+    <!-- <inertia ixx="0.5" ixy="0" ixz="0" iyy="0.5" iyz="0" izz="0.5" /> -->
+    <inertia ixx="0.25925" ixy="0" ixz="0" iyy="0.32216" iyz="0" izz="0.52516" />
     </inertial>
  </link>
@@ -108,5 +110,5 @@
       <mass value="1" />
       <origin xyz="-0.15 0.15 -0.05" rpy="-1.57 0.0 0.0"/>
-      <inertia ixx="0.1" ixy="0" ixz="0" iyy="0.1" iyz="0" izz="0.1" />
+      <inertia ixx="0.001" ixy="0" ixz="0" iyy="0.002" iyz="0" izz="0.001" />
     </inertial>
   </link>
@@ -118,4 +120,5 @@
     <axis xyz="0 0 1"/>
     <limit effort="100" velocity="100.0"  lower="-5000" upper="5000" />
+    <dynamics damping="0.1"/>
   </joint>
   <!--link name="visual_right_wheel">
@@ -150,5 +153,5 @@
       <mass value="1" />
        <origin xyz="-0.15 0.15 -0.05" rpy="-1.57 0.0 0.0"/>
-      <inertia ixx="0.1" ixy="0" ixz="0" iyy="0.1" iyz="0" izz="0.1" />
+      <inertia ixx="0.001" ixy="0" ixz="0" iyy="0.002" iyz="0" izz="0.001" />
     </inertial>
   </link>
@@ -161,8 +164,12 @@
     <axis xyz="0 0 1"/>
     <limit effort="100" velocity="100.0"  lower="-5000" upper="5000" />
+    <dynamics damping="0.1"/>
   </joint>
   <xacro:sensor_hokuyo name="hokuyo" parent="base_link" size="0.05 0.05 0.05">
     <origin xyz="0.25 0 0.1" rpy="0 0 0"/>
   </xacro:sensor_hokuyo>
+  <xacro:caster sub="0" parent="base_link" transX="0.15" transY="0.0" transZ="-0.075" />
+    <!-- <origin xyz="0.25 0 0.1" rpy="0 0 0"/> -->
+  <!-- </xacro:caster> -->
   <transmission name="tran1">
     <type>transmission_interface/SimpleTransmission</type>

Commit message: update

File: orne_description/urdf/gamma/orne_gamma.urdf.xacro (robot description, xacro)
@@ -1,5 +1,5 @@
 <?xml version="1.0"?>
 <!-- Revolute-Revolute Manipulator -->
-<robot name="orne_gamma" xmlns:xacro="http://www.ros.org/wiki/xacro">
+<robot name="orne_gamma" xmlns:xacro="http://ros.org/wiki/xacro">
   <!-- Constants for robot dimensions -->
   <xacro:property name="PI" value="3.1415926535897931"/>
@@ -97,4 +97,6 @@
     <collision name="collision">
       <!-- <origin xyz="0 0.0 -0.10" rpy="0 1.5707 1.5707"/> -->
+      <!-- <origin xyz="-0.15 0.15 -0.05" rpy="-1.57 0.0 0.0"/> -->
+      <origin xyz="0.0 0.0 0.0" rpy="0.0 0.0 0.0"/>
       <geometry>
          <cylinder  length="0.03" radius="0.0725"/>
@@ -103,4 +105,6 @@
     <visual name="visual">
       <!-- <origin xyz="0 0.0 -0.10" rpy="0 0 0"/> -->
+      <!-- <origin xyz="-0.15 0.15 -0.05" rpy="-1.57 0.0 0.0"/> -->
+      <origin xyz="0.0 0.0 0.0" rpy="0.0 0.0 0.0"/>
       <geometry>
         <cylinder  length="0.03" radius="0.0725"/>
@@ -109,5 +113,6 @@
     <inertial>
       <mass value="1" />
-      <origin xyz="-0.15 0.15 -0.05" rpy="-1.57 0.0 0.0"/>
+      <!-- <origin xyz="-0.15 0.15 -0.05" rpy="-1.57 0.0 0.0"/> -->
+      <origin xyz="0.0 0.0 0.0" rpy="0.0 0.0 0.0"/>
       <inertia ixx="0.001" ixy="0" ixz="0" iyy="0.002" iyz="0" izz="0.001" />
     </inertial>
@@ -138,4 +143,6 @@
   <link name="right_wheel">
     <collision name="collision">
+      <!-- <origin xyz="-0.15 -0.15 -0.05" rpy="-1.57 0.0 0.0"/> -->
+      <origin xyz="0.0 0.0 0.0" rpy="0.0 0.0 0.0"/>
       <!-- <origin xyz="0 0.0 -0.10" rpy="0 1.5707 1.5707"/> -->
       <!-- <origin xyz="0 0.15 -0.05" rpy="1.57 0 0"/> -->
@@ -146,4 +153,6 @@
     <visual name="visual">
       <!-- <origin xyz="0 0.0 -0.10" rpy="0 1.5707 1.5707"/> -->
+      <!-- <origin xyz="-0.15 -0.15 -0.05" rpy="-1.57 0.0 0.0"/> -->
+      <origin xyz="0.0 0.0 0.0" rpy="0.0 0.0 0.0"/>
       <geometry>
         <cylinder  length="0.03" radius="0.0725"/>
@@ -152,5 +161,6 @@
     <inertial>
       <mass value="1" />
-       <origin xyz="-0.15 0.15 -0.05" rpy="-1.57 0.0 0.0"/>
+      <!-- <origin xyz="-0.15 -0.15 -0.05" rpy="-1.57 0.0 0.0"/> -->
+      <origin xyz="0.0 0.0 0.0" rpy="0.0 0.0 0.0"/>
       <inertia ixx="0.001" ixy="0" ixz="0" iyy="0.002" iyz="0" izz="0.001" />
     </inertial>
@@ -192,3 +202,52 @@
     </actuator>
   </transmission>
+  <joint name="camera_joint" type="fixed">
+    <origin xyz="0.223 -0.011 0.565" rpy="0 0.124 0"/>
+    <parent link="base_link"/>
+    <child link="camera_link"/>
+  </joint>
+  <link name="camera_link">
+    <collision>
+      <origin xyz="0.005 0.011 0.013" rpy="0 0 0"/>
+      <geometry>
+        <box size="0.015 0.030 0.027"/>
+      </geometry>
+    </collision>
+  </link>
+  <joint name="camera_rgb_joint" type="fixed">
+    <origin xyz="0.003 0.011 0.009" rpy="0 0 0"/>
+    <parent link="camera_link"/>
+    <child link="camera_rgb_frame"/>
+  </joint>
+  <link name="camera_rgb_frame"/>
+  <joint name="camera_rgb_optical_joint" type="fixed">
+    <origin xyz="0 0 0" rpy="-1.57 0 -1.57"/>
+    <parent link="camera_rgb_frame"/>
+    <child link="camera_rgb_optical_frame"/>
+  </joint>
+  <link name="camera_rgb_optical_frame"/>
+  <joint name="camera_rgb_left_joint" type="fixed">
+    <origin xyz="0.003 0.111 0.009" rpy="0 0 0.175"/>
+    <parent link="camera_link"/>
+    <child link="camera_rgb_left_frame"/>
+  </joint>
+  <link name="camera_rgb_left_frame"/>
+  <joint name="camera_rgb_optical_left_joint" type="fixed">
+    <origin xyz="0 0 0" rpy="-1.57 0 -1.57"/>
+    <parent link="camera_rgb_left_frame"/>
+    <child link="camera_rgb_optical_left_frame"/>
+  </joint>
+  <link name="camera_rgb_optical_left_frame"/>
+  <joint name="camera_rgb_right_joint" type="fixed">
+    <origin xyz="0.003 -0.089 0.009" rpy="0 0 -0.175"/>
+    <parent link="camera_link"/>
+    <child link="camera_rgb_right_frame"/>
+  </joint>
+  <link name="camera_rgb_right_frame"/>
+  <joint name="camera_rgb_optical_right_joint" type="fixed">
+    <origin xyz="0 0 0" rpy="-1.57 0 -1.57"/>
+    <parent link="camera_rgb_right_frame"/>
+    <child link="camera_rgb_optical_right_frame"/>
+  </joint>
+  <link name="camera_rgb_optical_right_frame"/>
 </robot>

File: orne_description/urdf/gamma/orne_gamma_caster_fix.urdf.xacro (robot description, xacro)
@@ -2,5 +2,5 @@
 <robot name="caster" xmlns:xacro="http://www.ros.org/wiki/xacro">
   <!-- Casters -->
-  <xacro:property name="caster_radius" value="0.042650" /> <!-- in m -->
+  <xacro:property name="caster_radius" value="0.05250" /> <!-- in m -->
   <xacro:property name="caster_mass"   value="1.00" /> <!-- in kg-->
   <xacro:macro name="caster" params="sub parent transX transY transZ">
